Commit message: Update robot.urdf

File: cleanbit_control/model/robot.urdf (robot description, URDF)
Before this commit: robot differential_drive_robot, 5 links, 4 joints
Links:
- removed link caster_link
- added link front_marker_link; visual box size=0.04 0.22 0.03
- added link left_track_link, mass 1; collision box size=0.42 0.055 0.045; visual box size=0.42 0.055 0.045
- added link rear_left_wheel_link, mass 1; collision cylinder length=0.05 radius=0.1; visual cylinder length=0.05 radius=0.1
- added link rear_right_wheel_link, mass 1; collision cylinder length=0.05 radius=0.1; visual cylinder length=0.05 radius=0.1
- added link right_track_link, mass 1; collision box size=0.42 0.055 0.045; visual box size=0.42 0.055 0.045
- link laser_frame: mass 2 -> 0.5; geometry collision cylinder length=0.05 radius=0.08; visual cylinder length=0.05 radius=0.08
Joints:
- removed joint caster_joint
- added joint front_marker_joint: type fixed, parent body_link, child front_marker_link, origin xyz=0.27 0 0.03 rpy=0 0 0
- added joint left_track_joint: type fixed, parent body_link, child left_track_link, origin xyz=0 0.175 -0.05 rpy=0 0 0
- added joint rear_left_wheel_joint: type fixed, parent body_link, child rear_left_wheel_link, origin xyz=-0.15 0.175 -0.05 rpy=0 0 0
- added joint rear_right_wheel_joint: type fixed, parent body_link, child rear_right_wheel_link, origin xyz=-0.15 -0.175 -0.05 rpy=0 0 0
- added joint right_track_joint: type fixed, parent body_link, child right_track_link, origin xyz=0 -0.175 -0.05 rpy=0 0 0
- joint laser_joint: origin xyz=0.1 0 0.175 rpy=0 0 0 -> xyz=0.18 0 0.175 rpy=0 0 0
- joint left_wheel_joint: origin xyz=-0.15 0.175 -0.05 rpy=0 0 0 -> xyz=0.15 0.175 -0.05 rpy=0 0 0
- joint right_wheel_joint: origin xyz=-0.15 -0.175 -0.05 rpy=0 0 0 -> xyz=0.15 -0.175 -0.05 rpy=0 0 0
