Commit message: Update robot.xacro

File: cleanbit_control/model/robot.xacro (robot description, xacro)
@@ -1,10 +1,18 @@
 <?xml version="1.0"?>
-<robot name="spazz.ino" xmlns:xacro="http://www.ros.org/wiki/xacro">
+<robot name="spazzino" xmlns:xacro="http://www.ros.org/wiki/xacro">
+    <!-- ========================================================= -->
     <!-- Robot Parameters -->
+    <!-- Convenzione ROS:
+         X = avanti
+         Y = sinistra
+         Z = alto
+         In questo modello:
+         davanti = lato ruote motrici
+    ========================================================== -->
     <xacro:property name="PI" value="3.14159265"/>
     <xacro:property name="body_length" value="0.24"/>
     <xacro:property name="body_width" value="0.2"/>
     <xacro:property name="body_height" value="0.165"/>
-    <xacro:property name="body_density" value="7850.0"/> <!-- Steel -->
+    <xacro:property name="body_density" value="7850.0"/>
     <xacro:property name="body_mass" value="${body_density * body_length * body_height * body_width}"/>
     <xacro:property name="body_inertia_x" value="${1.0/12.0 * body_mass * (body_height*body_height + body_width*body_width)}"/>
@@ -15,20 +23,39 @@
     <xacro:property name="wheel_separation" value="${body_width + wheel_width}"/>
     <xacro:property name="wheel_offset" value="${body_length/2 - wheel_radius}"/>
-    <xacro:property name="wheel_density" value="900"/> <!-- Ruber -->
+    <xacro:property name="wheel_density" value="900"/>
     <xacro:property name="wheel_mass" value="${wheel_density * PI * wheel_radius * wheel_radius * wheel_width}"/>
     <xacro:property name="wheel_inertia_x" value="${1.0/12.0 * wheel_mass * (3*wheel_radius*wheel_radius + wheel_width*wheel_width)}"/>
     <xacro:property name="wheel_inertia_y" value="${1.0/12.0 * wheel_mass * (3*wheel_radius*wheel_radius + wheel_width*wheel_width)}"/>
     <xacro:property name="wheel_inertia_z" value="${1.0/2.0 * wheel_mass * wheel_radius * wheel_radius}"/>
-    <xacro:property name="caster_radius" value="0.055"/>
-    <xacro:property name="caster_offset" value="${body_length/2 - caster_radius}"/>
-    <xacro:property name="caster_density" value="0.1"/>
-    <xacro:property name="caster_mass" value="${caster_density * 4.0/3.0 * PI * caster_radius * caster_radius * caster_radius}"/>
-    <xacro:property name="caster_inertia_x" value="${2.0/5.0 * caster_mass * caster_radius * caster_radius}"/>
-    <xacro:property name="caster_inertia_y" value="${2.0/5.0 * caster_mass * caster_radius * caster_radius}"/>
-    <xacro:property name="caster_inertia_z" value="${2.0/5.0 * caster_mass * caster_radius * caster_radius}"/>
+    <xacro:property name="track_length" value="${body_length}"/>
+    <xacro:property name="track_width" value="0.035"/>
+    <xacro:property name="track_height" value="0.035"/>
+    <xacro:property name="laser_radius" value="0.04"/>
+    <xacro:property name="laser_height" value="0.035"/>
     <!-- Control Parameters -->
     <xacro:property name="max_linear_acceleration" value="10"/>
-    <!-- Links -->
+    <!-- ========================================================= -->
+    <!-- Materials -->
+    <!-- ========================================================= -->
+    <material name="body_material">
+        <color rgba="0.25 0.25 0.25 1.0"/>
+    </material>
+    <material name="wheel_material">
+        <color rgba="0.0 0.0 0.0 1.0"/>
+    </material>
+    <material name="track_material">
+        <color rgba="0.02 0.02 0.02 1.0"/>
+    </material>
+    <material name="laser_material">
+        <color rgba="1.0 0.0 0.0 1.0"/>
+    </material>
+    <material name="front_marker_material">
+        <color rgba="0.0 0.8 1.0 1.0"/>
+    </material>
+    <!-- ========================================================= -->
     <!-- Body Link -->
+    <!-- body_link è il frame principale del robot.
+         X positivo = davanti, cioè lato ruote motrici.
+    ========================================================== -->
     <link name="body_link">
         <visual>
@@ -37,7 +64,5 @@
                 <box size="${body_length} ${body_width} ${body_height}"/>
             </geometry>
-            <material name="body_material">
-                <color rgba="0.25 0.25 0.25 1.0"/>
-            </material>
+            <material name="body_material"/>
         </visual>
         <collision>
@@ -49,9 +74,17 @@
         <inertial>
             <mass value="10"/>
-            <inertia ixx="${body_inertia_x}" ixy="0.0" ixz="0.0" iyy="${body_inertia_y}" iyz="0" izz="${body_inertia_z}"/>
+            <inertia
+                ixx="${body_inertia_x}" ixy="0.0" ixz="0.0"
+                iyy="${body_inertia_y}" iyz="0.0"
+                izz="${body_inertia_z}"/>
             <origin xyz="0 0 0.027" rpy="0 0 0"/>
         </inertial>
     </link>
+    <!-- ========================================================= -->
     <!-- Base Footprint -->
+    <!-- Frame a terra usato spesso da Nav2/RViz.
+         Lo lascio collegato a body_link.
+    ========================================================== -->
+    <link name="base_footprint"/>
     <joint name="base_footprint_joint" type="fixed">
         <parent link="body_link"/>
@@ -59,7 +92,28 @@
         <origin xyz="0 0 0" rpy="0 0 0"/>
     </joint>
-    <link name="base_footprint">
-    </link>
-    <!-- Left Wheel -->
+    <!-- ========================================================= -->
+    <!-- Front Marker -->
+    <!-- Piccolo marker davanti per vedere subito il muso in RViz.
+         È sul lato +X.
+    ========================================================== -->
+    <link name="front_marker_link">
+        <visual>
+            <origin xyz="0 0 0" rpy="0 0 0"/>
+            <geometry>
+                <box size="0.015 0.14 0.025"/>
+            </geometry>
+            <material name="front_marker_material"/>
+        </visual>
+    </link>
+    <joint name="front_marker_joint" type="fixed">
+        <parent link="body_link"/>
+        <child link="front_marker_link"/>
+        <origin xyz="${body_length/2 + 0.012} 0 0.11" rpy="0 0 0"/>
+    </joint>
+    <!-- ========================================================= -->
+    <!-- Left Drive Wheel -->
+    <!-- Ruota motrice sinistra DAVANTI.
+         X positivo perché davanti = lato ruote motrici.
+    ========================================================== -->
     <link name="left_wheel_link">
         <visual>
@@ -68,119 +122,240 @@
                 <cylinder radius="${wheel_radius}" length="${wheel_width}"/>
             </geometry>
-            <material name="wheel_material">
-                <color rgba="0.0 0.0 0.0 1.0"/>
-            </material>
-        </visual>
-        <collision>
-            <origin xyz="0.0 0.0 0.0" rpy="1.570795 0.0 0.0"/>
-            <geometry>
-                <cylinder radius="${wheel_radius}" length="${wheel_width}"/>
-            </geometry>
-        </collision>
-        <inertial>
-            <mass value="2"/>
-            <inertia ixx="${wheel_inertia_x}" ixy="0.0" ixz="0.0" iyy="${wheel_inertia_y}" iyz="0" izz="${wheel_inertia_z}"/>
-            <origin xyz="0.0 0.0 0.0" rpy="1.570795 0.0 0.0"/>
-        </inertial>
-    </link>
-    <!-- Right Wheel -->
-    <link name="right_wheel_link">
-        <visual>
-            <origin xyz="0.0 0.0 0.0" rpy="1.570795 0.0 0.0"/>
-            <geometry>
-                <cylinder radius="${wheel_radius}" length="${wheel_width}"/>
-            </geometry>
-            <material name="wheel_material">
-                <color rgba="0.0 0.0 0.0 1.0"/>
-            </material>
-        </visual>
-        <collision>
-            <origin xyz="0.0 0.0 0.0" rpy="1.570795 0.0 0.0"/>
-            <geometry>
-                <cylinder radius="${wheel_radius}" length="${wheel_width}"/>
-            </geometry>
-        </collision>
-        <inertial>
-            <mass value="2"/>
-            <inertia ixx="${wheel_inertia_x}" ixy="0.0" ixz="0.0" iyy="${wheel_inertia_y}" iyz="0" izz="${wheel_inertia_z}"/>
-            <origin xyz="0.0 0.0 0.0" rpy="1.570795 0.0 0.0"/>
-        </inertial>
-    </link>
-    <!-- Caster Wheel -->
-    <link name="caster_link">
-        <visual>
-            <origin xyz="0.0 0.0 0.0" rpy="0.0 0.0 0.0"/>
-            <geometry>
-                <sphere radius="${caster_radius}"/>
-            </geometry>
-            <material name="caster_material">
-                <color rgba="0.0 0.0 0.0 1.0"/>
-            </material>
-        </visual>
-        <collision>
-            <origin xyz="0.0 0.0 0.0" rpy="0.0 0.0 0.0"/>
-            <geometry>
-                <sphere radius="${caster_radius}"/>
-            </geometry>
-        </collision>
-        <inertial>
-            <mass value="0.5"/>
-            <inertia ixx="${caster_inertia_x}" ixy="0.0" ixz="0.0" iyy="${caster_inertia_y}" iyz="0" izz="${caster_inertia_z}"/>
-            <origin xyz="0 0 0" rpy="0 0 0"/>
-        </inertial>
-    </link>
-    <!-- LIDAR -->
-    <link name="laser_frame">
-        <visual>
-            <origin xyz="0.0 0.0 0.0" rpy="0.0 0.0 0.0"/>
-            <geometry>
-                <cylinder radius="${wheel_radius}" length="${wheel_width}"/>
-            </geometry>
-            <material name="wheel_material">
-                <color rgba="1.0 0.0 0.0 0.0"/>
-            </material>
-        </visual>
-        <collision>
-            <origin xyz="0.0 0.0 0.0" rpy="0.0 0.0 0.0"/>
-            <geometry>
-                <cylinder radius="${wheel_radius}" length="${wheel_width}"/>
-            </geometry>
-        </collision>
-        <inertial>
-            <mass value="2"/>
-            <inertia ixx="${wheel_inertia_x}" ixy="0.0" ixz="0.0" iyy="${wheel_inertia_y}" iyz="0" izz="${wheel_inertia_z}"/>
-            <origin xyz="0.0 0.0 0.0" rpy="0.0 0.0 0.0"/>
-        </inertial>
-    </link>
-    <!-- Joints -->
-    <!-- Left Wheel Joint -->
+            <material name="wheel_material"/>
+        </visual>
+        <collision>
+            <origin xyz="0.0 0.0 0.0" rpy="1.570795 0.0 0.0"/>
+            <geometry>
+                <cylinder radius="${wheel_radius}" length="${wheel_width}"/>
+            </geometry>
+        </collision>
+        <inertial>
+            <mass value="${wheel_mass}"/>
+            <inertia
+                ixx="${wheel_inertia_x}" ixy="0.0" ixz="0.0"
+                iyy="${wheel_inertia_y}" iyz="0.0"
+                izz="${wheel_inertia_z}"/>
+            <origin xyz="0.0 0.0 0.0" rpy="1.570795 0.0 0.0"/>
+        </inertial>
+    </link>
     <joint name="left_wheel_joint" type="continuous">
-        <origin xyz="-${wheel_offset} ${wheel_separation/2} -${wheel_radius/2}" rpy="0 0 0"/>
         <parent link="body_link"/>
         <child link="left_wheel_link"/>
+        <!-- Prima era -${wheel_offset}; ora è +${wheel_offset} -->
+        <origin xyz="${wheel_offset} ${wheel_separation/2} -${wheel_radius/2}" rpy="0 0 0"/>
         <axis xyz="0 1 0"/>
         <limit effort="100" velocity="10.0"/>
         <dynamics damping="0.1" friction="0.1"/>
     </joint>
-    <!-- Right Wheel Joint -->
+    <!-- ========================================================= -->
+    <!-- Right Drive Wheel -->
+    <!-- Ruota motrice destra DAVANTI.
+    ========================================================== -->
+    <link name="right_wheel_link">
+        <visual>
+            <origin xyz="0.0 0.0 0.0" rpy="1.570795 0.0 0.0"/>
+            <geometry>
+                <cylinder radius="${wheel_radius}" length="${wheel_width}"/>
+            </geometry>
+            <material name="wheel_material"/>
+        </visual>
+        <collision>
+            <origin xyz="0.0 0.0 0.0" rpy="1.570795 0.0 0.0"/>
+            <geometry>
+                <cylinder radius="${wheel_radius}" length="${wheel_width}"/>
+            </geometry>
+        </collision>
+        <inertial>
+            <mass value="${wheel_mass}"/>
+            <inertia
+                ixx="${wheel_inertia_x}" ixy="0.0" ixz="0.0"
+                iyy="${wheel_inertia_y}" iyz="0.0"
+                izz="${wheel_inertia_z}"/>
+            <origin xyz="0.0 0.0 0.0" rpy="1.570795 0.0 0.0"/>
+        </inertial>
+    </link>
     <joint name="right_wheel_joint" type="continuous">
-        <origin xyz="-${wheel_offset} ${-wheel_separation/2} -${wheel_radius/2}" rpy="0 0 0"/>
         <parent link="body_link"/>
         <child link="right_wheel_link"/>
+        <!-- Prima era -${wheel_offset}; ora è +${wheel_offset} -->
+        <origin xyz="${wheel_offset} ${-wheel_separation/2} -${wheel_radius/2}" rpy="0 0 0"/>
         <axis xyz="0 1 0"/>
         <limit effort="100" velocity="10.0"/>
         <dynamics damping="0.1" friction="0.1"/>
     </joint>
-    <!-- Caster Wheel Joint (fixed) -->
-    <joint name="caster_joint" type="fixed">
-        <origin xyz="${caster_offset} 0 -${caster_radius/2}" rpy="0 0 0"/>
-        <parent link="body_link"/>
-        <child link="caster_link"/>
-    </joint>
+    <!-- ========================================================= -->
+    <!-- Rear Left Wheel -->
+    <!-- Ruota posteriore sinistra, solo visiva/fissa.
+         Sostituisce il caster.
+    ========================================================== -->
+    <link name="rear_left_wheel_link">
+        <visual>
+            <origin xyz="0.0 0.0 0.0" rpy="1.570795 0.0 0.0"/>
+            <geometry>
+                <cylinder radius="${wheel_radius}" length="${wheel_width}"/>
+            </geometry>
+            <material name="wheel_material"/>
+        </visual>
+        <collision>
+            <origin xyz="0.0 0.0 0.0" rpy="1.570795 0.0 0.0"/>
+            <geometry>
+                <cylinder radius="${wheel_radius}" length="${wheel_width}"/>
+            </geometry>
+        </collision>
+        <inertial>
+            <mass value="${wheel_mass}"/>
+            <inertia
+                ixx="${wheel_inertia_x}" ixy="0.0" ixz="0.0"
+                iyy="${wheel_inertia_y}" iyz="0.0"
+                izz="${wheel_inertia_z}"/>
+            <origin xyz="0.0 0.0 0.0" rpy="1.570795 0.0 0.0"/>
+        </inertial>
+    </link>
+    <joint name="rear_left_wheel_joint" type="fixed">
+        <parent link="body_link"/>
+        <child link="rear_left_wheel_link"/>
+        <!-- Dietro = X negativo -->
+        <origin xyz="-${wheel_offset} ${wheel_separation/2} -${wheel_radius/2}" rpy="0 0 0"/>
+    </joint>
+    <!-- ========================================================= -->
+    <!-- Rear Right Wheel -->
+    <!-- Ruota posteriore destra, solo visiva/fissa.
+    ========================================================== -->
+    <link name="rear_right_wheel_link">
+        <visual>
+            <origin xyz="0.0 0.0 0.0" rpy="1.570795 0.0 0.0"/>
+            <geometry>
+                <cylinder radius="${wheel_radius}" length="${wheel_width}"/>
+            </geometry>
+            <material name="wheel_material"/>
+        </visual>
+        <collision>
+            <origin xyz="0.0 0.0 0.0" rpy="1.570795 0.0 0.0"/>
+            <geometry>
+                <cylinder radius="${wheel_radius}" length="${wheel_width}"/>
+            </geometry>
+        </collision>
+        <inertial>
+            <mass value="${wheel_mass}"/>
+            <inertia
+                ixx="${wheel_inertia_x}" ixy="0.0" ixz="0.0"
+                iyy="${wheel_inertia_y}" iyz="0.0"
+                izz="${wheel_inertia_z}"/>
+            <origin xyz="0.0 0.0 0.0" rpy="1.570795 0.0 0.0"/>
+        </inertial>
+    </link>
+    <joint name="rear_right_wheel_joint" type="fixed">
+        <parent link="body_link"/>
+        <child link="rear_right_wheel_link"/>
+        <!-- Dietro = X negativo -->
+        <origin xyz="-${wheel_offset} ${-wheel_separation/2} -${wheel_radius/2}" rpy="0 0 0"/>
+    </joint>
+    <!-- ========================================================= -->
+    <!-- Left Track Visual -->
+    <!-- Cingolo sinistro visivo.
+         Non è una ruota motrice fisica per il plugin/controllo,
+         serve a rappresentare meglio il robot.
+    ========================================================== -->
+    <link name="left_track_link">
+        <visual>
+            <origin xyz="0 0 0" rpy="0 0 0"/>
+            <geometry>
+                <box size="${track_length} ${track_width} ${track_height}"/>
+            </geometry>
+            <material name="track_material"/>
+        </visual>
+        <collision>
+            <origin xyz="0 0 0" rpy="0 0 0"/>
+            <geometry>
+                <box size="${track_length} ${track_width} ${track_height}"/>
+            </geometry>
+        </collision>
+        <inertial>
+            <mass value="0.5"/>
+            <inertia
+                ixx="0.001" ixy="0.0" ixz="0.0"
+                iyy="0.001" iyz="0.0"
+                izz="0.001"/>
+            <origin xyz="0 0 0" rpy="0 0 0"/>
+        </inertial>
+    </link>
+    <joint name="left_track_joint" type="fixed">
+        <parent link="body_link"/>
+        <child link="left_track_link"/>
+        <origin xyz="0 ${wheel_separation/2} -${wheel_radius/2}" rpy="0 0 0"/>
+    </joint>
+    <!-- ========================================================= -->
+    <!-- Right Track Visual -->
+    <!-- Cingolo destro visivo.
+    ========================================================== -->
+    <link name="right_track_link">
+        <visual>
+            <origin xyz="0 0 0" rpy="0 0 0"/>
+            <geometry>
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