Commit message: Update robot.xacro

File: cleanbit_control/model/robot.xacro (robot description, xacro)
@@ -7,6 +7,6 @@
          Y = sinistra
          Z = alto
-         In questo modello:
-         davanti = lato ruote motrici
+         base_link è il frame principale corretto.
+         body_link è la geometria ruotata di 180 gradi rispetto a base_link.
     ========================================================== -->
     <xacro:property name="PI" value="3.14159265"/>
@@ -33,5 +33,4 @@
     <xacro:property name="laser_radius" value="0.04"/>
     <xacro:property name="laser_height" value="0.035"/>
-    <!-- Control Parameters -->
     <xacro:property name="max_linear_acceleration" value="10"/>
     <!-- ========================================================= -->
@@ -54,7 +53,17 @@
     </material>
     <!-- ========================================================= -->
-    <!-- Body Link -->
-    <!-- body_link è il frame principale del robot.
-         X positivo = davanti, cioè lato ruote motrici.
+    <!-- BASE LINK -->
+    <!-- Questo è il frame principale ROS.
+         In RViz devi guardare questo:
+         X rosso = avanti reale del robot
+         Y verde = sinistra
+         Z blu = alto
+    ========================================================== -->
+    <link name="base_link"/>
+    <!-- ========================================================= -->
+    <!-- BODY LINK -->
+    <!-- Geometria del corpo.
+         Viene ruotata di 180 gradi rispetto a base_link
+         tramite base_to_body_joint.
     ========================================================== -->
     <link name="body_link">
@@ -82,11 +91,21 @@
     </link>
     <!-- ========================================================= -->
+    <!-- BASE TO BODY JOINT -->
+    <!-- Questa è la correzione dei 180 gradi.
+         base_link rimane corretto.
+         body_link viene girato.
+    ========================================================== -->
+    <joint name="base_to_body_joint" type="fixed">
+        <parent link="base_link"/>
+        <child link="body_link"/>
+        <origin xyz="0 0 0" rpy="0 0 ${PI}"/>
+    </joint>
+    <!-- ========================================================= -->
     <!-- Base Footprint -->
-    <!-- Frame a terra usato spesso da Nav2/RViz.
-         Lo lascio collegato a body_link.
+    <!-- Frame a terra collegato a base_link, non a body_link.
     ========================================================== -->
     <link name="base_footprint"/>
     <joint name="base_footprint_joint" type="fixed">
-        <parent link="body_link"/>
+        <parent link="base_link"/>
         <child link="base_footprint"/>
         <origin xyz="0 0 0" rpy="0 0 0"/>
@@ -94,6 +113,7 @@
     <!-- ========================================================= -->
     <!-- Front Marker -->
-    <!-- Piccolo marker davanti per vedere subito il muso in RViz.
-         È sul lato +X.
+    <!-- Marker davanti rispetto al body_link.
+         Siccome body_link è ruotato di PI rispetto a base_link,
+         questo marker serve solo come riferimento visivo del modello.
     ========================================================== -->
     <link name="front_marker_link">
@@ -113,6 +133,6 @@
     <!-- ========================================================= -->
     <!-- Left Drive Wheel -->
-    <!-- Ruota motrice sinistra DAVANTI.
-         X positivo perché davanti = lato ruote motrici.
+    <!-- Ruota motrice sinistra.
+         Davanti del modello body_link: X positivo.
     ========================================================== -->
     <link name="left_wheel_link">
@@ -142,5 +162,4 @@
         <parent link="body_link"/>
         <child link="left_wheel_link"/>
-        <!-- Prima era -${wheel_offset}; ora è +${wheel_offset} -->
         <origin xyz="${wheel_offset} ${wheel_separation/2} -${wheel_radius/2}" rpy="0 0 0"/>
         <axis xyz="0 1 0"/>
@@ -150,5 +169,5 @@
     <!-- ========================================================= -->
     <!-- Right Drive Wheel -->
-    <!-- Ruota motrice destra DAVANTI.
+    <!-- Ruota motrice destra.
     ========================================================== -->
     <link name="right_wheel_link">
@@ -178,5 +197,4 @@
         <parent link="body_link"/>
         <child link="right_wheel_link"/>
-        <!-- Prima era -${wheel_offset}; ora è +${wheel_offset} -->
         <origin xyz="${wheel_offset} ${-wheel_separation/2} -${wheel_radius/2}" rpy="0 0 0"/>
         <axis xyz="0 1 0"/>
@@ -186,6 +204,5 @@
     <!-- ========================================================= -->
     <!-- Rear Left Wheel -->
-    <!-- Ruota posteriore sinistra, solo visiva/fissa.
-         Sostituisce il caster.
+    <!-- Ruota posteriore sinistra, fissa/visiva.
     ========================================================== -->
     <link name="rear_left_wheel_link">
@@ -215,10 +232,9 @@
         <parent link="body_link"/>
         <child link="rear_left_wheel_link"/>
-        <!-- Dietro = X negativo -->
         <origin xyz="-${wheel_offset} ${wheel_separation/2} -${wheel_radius/2}" rpy="0 0 0"/>
     </joint>
     <!-- ========================================================= -->
     <!-- Rear Right Wheel -->
-    <!-- Ruota posteriore destra, solo visiva/fissa.
+    <!-- Ruota posteriore destra, fissa/visiva.
     ========================================================== -->
     <link name="rear_right_wheel_link">
@@ -248,5 +264,4 @@
         <parent link="body_link"/>
         <child link="rear_right_wheel_link"/>
-        <!-- Dietro = X negativo -->
         <origin xyz="-${wheel_offset} ${-wheel_separation/2} -${wheel_radius/2}" rpy="0 0 0"/>
     </joint>
@@ -254,6 +269,4 @@
     <!-- Left Track Visual -->
     <!-- Cingolo sinistro visivo.
-         Non è una ruota motrice fisica per il plugin/controllo,
-         serve a rappresentare meglio il robot.
     ========================================================== -->
     <link name="left_track_link">
@@ -319,13 +332,6 @@
     <!-- ========================================================= -->
     <!-- LIDAR -->
-    <!-- Lidar davanti, lato +X.
-         Il frame laser_frame deve avere:
-         X avanti
-         Y sinistra
-         Z alto
-         Se il LaserScan in RViz risulta ancora ruotato di 180°,
-         cambia solo il rpy del laser_joint da:
-         rpy="0 0 0"
-         a:
+    <!-- Lidar davanti rispetto al body_link.
+         Se il LaserScan risulta girato, modifica solo laser_joint:
          rpy="0 0 ${PI}"
     ========================================================== -->
@@ -356,5 +362,4 @@
         <parent link="body_link"/>
         <child link="laser_frame"/>
-        <!-- Lidar davanti: X positivo -->
         <origin xyz="${body_length/2 - 0.03} 0 0.125" rpy="0 0 0"/>
     </joint>

Commit message: Update robot.xacro

File: cleanbit_control/model/robot.xacro (robot description, xacro)
@@ -7,6 +7,6 @@
          Y = sinistra
          Z = alto
-         base_link è il frame principale corretto.
-         body_link è la geometria ruotata di 180 gradi rispetto a base_link.
+         Davanti reale del robot = lato ruote motrici + lidar.
+         Quindi ruote motrici e lidar stanno a X positivo.
     ========================================================== -->
     <xacro:property name="PI" value="3.14159265"/>
@@ -54,7 +54,6 @@
     <!-- ========================================================= -->
     <!-- BASE LINK -->
-    <!-- Questo è il frame principale ROS.
-         In RViz devi guardare questo:
-         X rosso = avanti reale del robot
+    <!-- Frame principale ROS:
+         X rosso = avanti reale
          Y verde = sinistra
          Z blu = alto
@@ -63,7 +62,6 @@
     <!-- ========================================================= -->
     <!-- BODY LINK -->
-    <!-- Geometria del corpo.
-         Viene ruotata di 180 gradi rispetto a base_link
-         tramite base_to_body_joint.
+    <!-- Corpo del robot.
+         NON viene più ruotato di 180 gradi.
     ========================================================== -->
     <link name="body_link">
@@ -92,16 +90,16 @@
     <!-- ========================================================= -->
     <!-- BASE TO BODY JOINT -->
-    <!-- Questa è la correzione dei 180 gradi.
-         base_link rimane corretto.
-         body_link viene girato.
+    <!-- Correzione importante:
+         prima era rpy="0 0 ${PI}", e quello girava tutto di 180°.
+         Ora è zero.
     ========================================================== -->
     <joint name="base_to_body_joint" type="fixed">
         <parent link="base_link"/>
         <child link="body_link"/>
-        <origin xyz="0 0 0" rpy="0 0 ${PI}"/>
-    </joint>
-    <!-- ========================================================= -->
-    <!-- Base Footprint -->
-    <!-- Frame a terra collegato a base_link, non a body_link.
+        <origin xyz="0 0 0" rpy="0 0 0"/>
+    </joint>
+    <!-- ========================================================= -->
+    <!-- BASE FOOTPRINT -->
+    <!-- Frame a terra collegato a base_link.
     ========================================================== -->
     <link name="base_footprint"/>
@@ -112,8 +110,6 @@
     </joint>
     <!-- ========================================================= -->
-    <!-- Front Marker -->
-    <!-- Marker davanti rispetto al body_link.
-         Siccome body_link è ruotato di PI rispetto a base_link,
-         questo marker serve solo come riferimento visivo del modello.
+    <!-- FRONT MARKER -->
+    <!-- Marker visivo sul davanti reale, cioè lato +X.
     ========================================================== -->
     <link name="front_marker_link">
@@ -132,7 +128,8 @@
     </joint>
     <!-- ========================================================= -->
-    <!-- Left Drive Wheel -->
-    <!-- Ruota motrice sinistra.
-         Davanti del modello body_link: X positivo.
+    <!-- LEFT DRIVE WHEEL -->
+    <!-- Ruota motrice sinistra DAVANTI.
+         X positivo = davanti.
+         Y positivo = sinistra.
     ========================================================== -->
     <link name="left_wheel_link">
@@ -168,6 +165,8 @@
     </joint>
     <!-- ========================================================= -->
-    <!-- Right Drive Wheel -->
-    <!-- Ruota motrice destra.
+    <!-- RIGHT DRIVE WHEEL -->
+    <!-- Ruota motrice destra DAVANTI.
+         X positivo = davanti.
+         Y negativo = destra.
     ========================================================== -->
     <link name="right_wheel_link">
@@ -203,5 +202,5 @@
     </joint>
     <!-- ========================================================= -->
-    <!-- Rear Left Wheel -->
+    <!-- REAR LEFT WHEEL -->
     <!-- Ruota posteriore sinistra, fissa/visiva.
     ========================================================== -->
@@ -235,5 +234,5 @@
     </joint>
     <!-- ========================================================= -->
-    <!-- Rear Right Wheel -->
+    <!-- REAR RIGHT WHEEL -->
     <!-- Ruota posteriore destra, fissa/visiva.
     ========================================================== -->
@@ -267,5 +266,5 @@
     </joint>
     <!-- ========================================================= -->
-    <!-- Left Track Visual -->
+    <!-- LEFT TRACK VISUAL -->
     <!-- Cingolo sinistro visivo.
     ========================================================== -->
@@ -299,5 +298,5 @@
     </joint>
     <!-- ========================================================= -->
-    <!-- Right Track Visual -->
+    <!-- RIGHT TRACK VISUAL -->
     <!-- Cingolo destro visivo.
     ========================================================== -->
@@ -332,6 +331,6 @@
     <!-- ========================================================= -->
     <!-- LIDAR -->
-    <!-- Lidar davanti rispetto al body_link.
-         Se il LaserScan risulta girato, modifica solo laser_joint:
+    <!-- Lidar davanti: X positivo.
+         Se il LaserScan risulta girato di 180°, ruota SOLO questo joint:
          rpy="0 0 ${PI}"
     ========================================================== -->
